File: gromofon.kicad_sch (KiCad schematic)
At the start: 17 parts, among them J1 power supply, J2 esp32, J3 TC4420, J4 flyback, Q1 IRFP260N, U1 L7812

Commit message: Add files via upload
Parts:
- removed C5: 10 µF, symbol Device:C
- added C5: 10 µF/50 V, symbol Device:C_Polarized
- C2: value 1 µF -> 1 µF / 50 V, X7R
- C3: value 10 nF/630 V -> 10 nF / 1000 V DC, MKP
- C4: value 100 nF -> 100 nF / 50 V, X7R
Connections:
- net +12V: now also C5.1
- net GND: now also C5.2
Other:
- moved on the sheet: C1, C2, C3, C4, D1, F1, J1, J2, J3, J4, Q1, R1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
